File: FTDI USB-Friend/ftdifriend-usb.sch (EAGLE design)
At the start: 20 parts, among them CN1 MINIB, CN2 MINIB, IC1 FT232RL

Commit message: small changes
Other:
- note removed: "CC Attrib & Share Alike"
- note removed: "FTDI Friend! A breakout board+ from adafruit.com"
Changed lines of the file:
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@@
 <?xml version="1.0" encoding="utf-8"?>
 <!DOCTYPE eagle SYSTEM "eagle.dtd">
-<eagle version="6.4">
+<eagle version="7.2.0">
 <drawing>
 <settings>
@@
 <sheet>
 <plain>
-<text x="101.6" y="-17.78" size="2.54" layer="94">CC Attrib &amp; Share Alike</text>
-<text x="101.6" y="-12.7" size="2.54" layer="94">FTDI Friend! A breakout board+ from adafruit.com</text>
 <text x="101.6" y="71.12" size="1.778" layer="97">CTS-&gt;GND</text>
 </plain>
